File: G491CC_Adaptor.kicad_pcb (KiCad board)
At the start: 2 copper layers, 33.5 x 31 mm, 26 parts, among them J1 Conn_01x12, J2 Conn_01x11, J3 Conn_01x11, J4 Conn_01x12, U1 STM32G491CCUx, U2 AP7343D-33W5, U3 TCR2EE33, Y1 ECX-1637B2 [10pF, 20MHz]

Commit message: LED resistor values
Parts:
- D1: value COLOR? -> RED
- D2: value COLOR? -> GREEN
- R1: value ? -> 205R
- R2: value ? -> 511R
Changed lines of the file:
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@@
       (effects (font (size 0.9 0.7) (thickness 0.155)))
     )
-    (fp_text value "?" (at 0 1.43) (layer "F.Fab")
+    (fp_text value "511R" (at 0 1.43) (layer "F.Fab")
       (effects (font (size 0.9 0.7) (thickness 0.155)))
     )
@@
       (effects (font (size 0.9 0.7) (thickness 0.155)))
     )
-    (fp_text value "COLOR?" (at 0 1.43) (layer "F.Fab")
+    (fp_text value "RED" (at 0 1.43) (layer "F.Fab")
       (effects (font (size 0.9 0.7) (thickness 0.155)))
     )
@@
       (effects (font (size 0.9 0.7) (thickness 0.155)))
     )
-    (fp_text value "?" (at 0 1.43) (layer "F.Fab")
+    (fp_text value "205R" (at 0 1.43) (layer "F.Fab")
       (effects (font (size 0.9 0.7) (thickness 0.155)))
     )
@@
       (effects (font (size 0.9 0.7) (thickness 0.155)))
     )
-    (fp_text value "COLOR?" (at 0 1.43) (layer "F.Fab")
-      (effects (font (size 0.9 0.7) (thickness 0.155)))
-    )
+    (fp_text value "GREEN" (at 0 1.43) (layer "F.Fab")
+      (effects (font (size 0.9 0.7) (thickness 0.155)))
+    )
